Commit message: Add: 7/4までのプログラム

File: mst110cr_description/urdf/mst110cr.urdf (robot description, URDF)
Before this commit: robot mst110cr, 6 links, 5 joints
Links:
- removed link mst110cr/base_link
- removed link mst110cr/body_link
- removed link mst110cr/track_link
- removed link mst110cr/vessel_cylinder_link
- removed link mst110cr/vessel_link
- removed link mst110cr/vessel_rod_link
- added link mst110cr_2/base_link
- added link mst110cr_2/body_link, mass 0.03; collision mesh filename=package://mst110cr_description/meshes/mst110cr-body.dae; visual mesh filename=package://mst110cr_description/meshes/mst110cr-body.dae
- added link mst110cr_2/track_link, mass 0.03; collision mesh filename=package://mst110cr_description/meshes/mst110cr-crawler.dae; visual mesh filename=package://mst110cr_description/meshes/mst110cr-crawler.dae
- added link mst110cr_2/vessel_cylinder_link, mass 0.03; collision mesh filename=package://mst110cr_description/meshes/mst110cr-vessel_cylin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; visual mesh filename=package://mst110cr_description/meshes/mst110cr-vessel_cylin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
- added link mst110cr_2/vessel_link, mass 0.03; collision mesh filename=package://mst110cr_description/meshes/mst110cr-vessel.dae; visual mesh filename=package://mst110cr_description/meshes/mst110cr-vessel.dae
- added link mst110cr_2/vessel_rod_link, mass 0.03; collision mesh filename=package://mst110cr_description/meshes/mst110cr-vessel_rod.d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; visual mesh filename=package://mst110cr_description/meshes/mst110cr-vessel_rod.d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
Joints:
- joint base_joint: child mst110cr/track_link -> mst110cr_2/track_link; parent mst110cr/base_link -> mst110cr_2/base_link
- joint swing_joint: child mst110cr/body_link -> mst110cr_2/body_link; parent mst110cr/track_link -> mst110cr_2/track_link
- joint vessel_cylinder_joint: child mst110cr/vessel_cylinder_link -> mst110cr_2/vessel_cylinder_link; parent mst110cr/body_link -> mst110cr_2/body_link
- joint vessel_pin_joint: child mst110cr/vessel_link -> mst110cr_2/vessel_link; parent mst110cr/body_link -> mst110cr_2/body_link
- joint vessel_rod_joint: child mst110cr/vessel_rod_link -> mst110cr_2/vessel_rod_link; parent mst110cr/vessel_cylinder_link -> mst110cr_2/vessel_cylinder_link

File: mst110cr_description/urdf/mst110cr.xacro (robot description, xacro)
@@ -2,11 +2,11 @@
 <robot name="mst110cr" xmlns:xacro="http://www.ros.org/wiki/xacro">
 	<!-- Base Link -->
-	<link name="mst110cr/base_link"/>
+	<link name="mst110cr_2/base_link"/>
 	<!-- Track {{{ -->
 	<joint name="base_joint" type="fixed">
-		<parent link="mst110cr/base_link"/>
-		<child link="mst110cr/track_link"/>
+		<parent link="mst110cr_2/base_link"/>
+		<child link="mst110cr_2/track_link"/>
 	</joint>
-	<link name="mst110cr/track_link">
+	<link name="mst110cr_2/track_link">
 		<visual>
 			<geometry>
@@ -32,8 +32,8 @@
 		<origin xyz="0 0 1"/>
 		<axis xyz="0 0 1"/>
-		<parent link="mst110cr/track_link"/>
-		<child link="mst110cr/body_link"/>
+		<parent link="mst110cr_2/track_link"/>
+		<child link="mst110cr_2/body_link"/>
 	</joint>
-	<link name="mst110cr/body_link">
+	<link name="mst110cr_2/body_link">
 		<visual>
 			<origin xyz="0 0 0"/>
@@ -61,9 +61,9 @@
 		<origin xyz="-2.389 0 0.562"/>
 		<axis xyz="0 1 0"/>
-		<parent link="mst110cr/body_link"/>
-		<child link="mst110cr/vessel_link"/>
+		<parent link="mst110cr_2/body_link"/>
+		<child link="mst110cr_2/vessel_link"/>
 		<limit lower="${radians(-60)}" upper="${radians(0)}" effort="500" velocity="6.159937255"/>
 	</joint>
-	<link name="mst110cr/vessel_link">
+	<link name="mst110cr_2/vessel_link">
 		<visual>
 			<origin xyz="0 0 0"/>
@@ -91,9 +91,9 @@
 		<origin xyz="-1.891 0 0.293"/>
 		<axis xyz="0 1 0"/>
-		<parent link="mst110cr/body_link"/>
-		<child link="mst110cr/vessel_cylinder_link"/>
+		<parent link="mst110cr_2/body_link"/>
+		<child link="mst110cr_2/vessel_cylinder_link"/>
 		<mimic joint="vessel_pin_joint" multiplier="${66/60}"/>
 	</joint>
-	<link name="mst110cr/vessel_cylinder_link">
+	<link name="mst110cr_2/vessel_cylinder_link">
 		<visual>
 			<origin xyz="0 0 0"/>
@@ -121,10 +121,10 @@
 		<origin xyz="0 0 0"/>
 		<axis xyz="1.039 0 0.282"/>
-		<parent link="mst110cr/vessel_cylinder_link"/>
-		<child link="mst110cr/vessel_rod_link"/>
+		<parent link="mst110cr_2/vessel_cylinder_link"/>
+		<child link="mst110cr_2/vessel_rod_link"/>
 		<limit lower="0" upper="0.6" effort="500" velocity="6.159937255"/>
 		<mimic joint="vessel_pin_joint" multiplier="${0.6/radians(-60)}"/>
 	</joint>
-	<link name="mst110cr/vessel_rod_link">
+	<link name="mst110cr_2/vessel_rod_link">
 		<visual>
 			<origin xyz="0 0 0"/>
