Commit message: Add: 正しいmst110crのモデルデータに差し替え

File: mst110cr_description/urdf/mst110cr.xacro (robot description, xacro)
@@ -1,36 +1,150 @@
 <?xml version="1.0"?>
-<robot xmlns:xacro="http://ros.org/wiki/xacro" name="simple_box">
-  <link name="base_link">
-    <inertial>
-      <origin xyz="0 0 1.625" rpy="0 0 0"/>
-      <mass value="16000.0"/>
-      <!-- 慣性モーメント（直方体 6.00×2.98×3.25 m, 16000 kg） -->
-      <!-- Ixx = 1/12*m*(b^2 + c^2) -->
-      <!-- Iyy = 1/12*m*(a^2 + c^2) -->
-      <!-- Izz = 1/12*m*(a^2 + b^2) -->
-      <inertia
-        ixx="25923.9333"
-        iyy="62083.3333"
-        izz="59840.5333"
-        ixy="0.0"
-        ixz="0.0"
-        iyz="0.0"/>
-    </inertial>
-    <visual>
-      <origin xyz="0 0 1.625" rpy="0 0 0"/>
-      <geometry>
-        <!-- 全長 6000 mm, 全幅 2980 mm, 全高 3250 mm -->
-        <box size="6.0 2.98 3.25"/>
-      </geometry>
-      <material name="Grey">
-        <color rgba="0.7 0.7 0.7 1.0"/>
-      </material>
-    </visual>
-    <collision>
-      <origin xyz="0 0 1.625" rpy="0 0 0"/>
-      <geometry>
-        <box size="6.0 2.98 3.25"/>
-      </geometry>
-    </collision>
-  </link>
+<robot name="mst110cr" xmlns:xacro="http://www.ros.org/wiki/xacro">
+	<!-- Base Link -->
+	<link name="mst110cr/base_link"/>
+	<!-- Track {{{ -->
+	<joint name="base_joint" type="fixed">
+		<parent link="mst110cr/base_link"/>
+		<child link="mst110cr/track_link"/>
+	</joint>
+	<link name="mst110cr/track_link">
+		<visual>
+			<geometry>
+				<mesh filename="package://mst110cr_description/meshes/mst110cr-crawler.dae"/>
+			</geometry>
+		</visual>
+		<collision>
+			<geometry>
+				<mesh filename="package://mst110cr_description/meshes/mst110cr-crawler.dae"/>
+			</geometry>
+		</collision>
+		<inertial>
+			<origin xyz="0 0 0" rpy="0 0 0"/>
+			<mass value="0.03"/>
+			<inertia ixx="1.0" ixy="0.0" ixz="0.0"
+								iyy="1.0" iyz="0.0"
+											izz="1.0"/>
+		</inertial>
+	</link>
+	<!-- }}} Track ends here -->
+	<!-- Body {{{ -->
+	<joint name="swing_joint" type="continuous">
+		<origin xyz="0 0 1"/>
+		<axis xyz="0 0 1"/>
+		<parent link="mst110cr/track_link"/>
+		<child link="mst110cr/body_link"/>
+	</joint>
+	<link name="mst110cr/body_link">
+		<visual>
+			<origin xyz="0 0 0"/>
+			<geometry>
+				<mesh filename="package://mst110cr_description/meshes/mst110cr-body.dae"/>
+			</geometry>
+		</visual>
+		<collision>
+			<origin xyz="0 0 0"/>
+			<geometry>
+				<mesh filename="package://mst110cr_description/meshes/mst110cr-body.dae"/>
+			</geometry>
+		</collision>
+		<inertial>
+			<origin xyz="0 0 0" rpy="0 0 0"/>
+			<mass value="0.03"/>
+			<inertia ixx="1.0" ixy="0.0" ixz="0.0"
+								iyy="1.0" iyz="0.0"
+											izz="1.0"/>
+		</inertial>
+	</link>
+	<!-- }}} Body ends here -->
+	<!-- Vessel {{{ -->
+	<joint name="vessel_pin_joint" type="revolute">
+		<origin xyz="-2.389 0 0.562"/>
+		<axis xyz="0 1 0"/>
+		<parent link="mst110cr/body_link"/>
+		<child link="mst110cr/vessel_link"/>
+		<limit lower="${radians(-60)}" upper="${radians(0)}" effort="500" velocity="6.159937255"/>
+	</joint>
+	<link name="mst110cr/vessel_link">
+		<visual>
+			<origin xyz="0 0 0"/>
+			<geometry>
+				<mesh filename="package://mst110cr_description/meshes/mst110cr-vessel.dae"/>
+			</geometry>
+		</visual>
+		<collision>
+			<origin xyz="0 0 0"/>
+			<geometry>
+				<mesh filename="package://mst110cr_description/meshes/mst110cr-vessel.dae"/>
+			</geometry>
+		</collision>
+		<inertial>
+			<origin xyz="0 0 0" rpy="0 0 0"/>
+			<mass value="0.03"/>
+			<inertia ixx="1.0" ixy="0.0" ixz="0.0"
+								iyy="1.0" iyz="0.0"
+											izz="1.0"/>
+		</inertial>
+	</link>
+	<!-- }}} Vessel ends here -->
+	<!-- Vessel Cylinder {{{ -->
+	<joint name="vessel_cylinder_joint" type="continuous">
+		<origin xyz="-1.891 0 0.293"/>
+		<axis xyz="0 1 0"/>
+		<parent link="mst110cr/body_link"/>
+		<child link="mst110cr/vessel_cylinder_link"/>
+		<mimic joint="vessel_pin_joint" multiplier="${66/60}"/>
+	</joint>
+	<link name="mst110cr/vessel_cylinder_link">
+		<visual>
+			<origin xyz="0 0 0"/>
+			<geometry>
+				<mesh filename="package://mst110cr_description/meshes/mst110cr-vessel_cylinder.dae"/>
+			</geometry>
+		</visual>
+		<collision>
+			<origin xyz="0 0 0"/>
+			<geometry>
+				<mesh filename="package://mst110cr_description/meshes/mst110cr-vessel_cylinder.dae"/>
+			</geometry>
+		</collision>
+		<inertial>
+			<origin xyz="0 0 0" rpy="0 0 0"/>
+			<mass value="0.03"/>
+			<inertia ixx="1.0" ixy="0.0" ixz="0.0"
+								iyy="1.0" iyz="0.0"
+											izz="1.0"/>
+		</inertial>
+	</link>
+	<!-- }}} Vessel Cylinder ends here -->
+	<!-- Vessel Rod {{{ -->
+	<joint name="vessel_rod_joint" type="prismatic">
+		<origin xyz="0 0 0"/>
+		<axis xyz="1.039 0 0.282"/>
+		<parent link="mst110cr/vessel_cylinder_link"/>
+		<child link="mst110cr/vessel_rod_link"/>
+		<limit lower="0" upper="0.6" effort="500" velocity="6.159937255"/>
+		<mimic joint="vessel_pin_joint" multiplier="${0.6/radians(-60)}"/>
+	</joint>
+	<link name="mst110cr/vessel_rod_link">
+		<visual>
+			<origin xyz="0 0 0"/>
+			<geometry>
+				<mesh filename="package://mst110cr_description/meshes/mst110cr-vessel_rod.dae"/>
+			</geometry>
+		</visual>
+		<collision>
+			<origin xyz="0 0 0"/>
+			<geometry>
+				<mesh filename="package://mst110cr_description/meshes/mst110cr-vessel_rod.dae"/>
+			</geometry>
+		</collision>
+		<inertial>
+			<origin xyz="0 0 0" rpy="0 0 0"/>
+			<mass value="0.03"/>
+			<inertia ixx="1.0" ixy="0.0" ixz="0.0"
+								iyy="1.0" iyz="0.0"
+											izz="1.0"/>
+		</inertial>
+	</link>
+	<!-- }}} Vessel Rod ends here -->
 </robot>

Commit message: add gnss_link to mst110cr.xacro

File: mst110cr_description/urdf/mst110cr.xacro (robot description, xacro)
@@ -148,3 +148,10 @@
 	</link>
 	<!-- }}} Vessel Rod ends here -->
+	<joint name="gnss_joint" type="fixed">
+		<origin xyz="1.42 0.60 2.20"/>
+		<axis xyz="0 0 1"/>
+		<parent link="mst110cr_2/body_link"/>
+		<child link="mst110cr_2/gnss_link"/>
+	</joint>
+	<link name="mst110cr_2/gnss_link"/>
 </robot>

Commit message: add livox and ouster link and joint

File: mst110cr_description/urdf/mst110cr.xacro (robot description, xacro)
@@ -57,4 +57,184 @@
 	</link>
 	<!-- }}} Body ends here -->
+	<!-- os_stand frame {{{ -->
+	<joint name="os_stand_joint" type="fixed">
+		<parent link="mst110cr_2/body_link"/>
+		<child link="mst110cr_2/os_stand"/>
+		<origin xyz="2.640 0.660 2.260" rpy="0 0 0"/>
+	</joint>
+	<link name="mst110cr_2/os_stand">
+		<visual>
+		<origin xyz="0 0 0"/>
+		<geometry>
+			<box size="0.01 0.01 0.01"/>
+		</geometry>
+		<material name="gray">
+			<color rgba="0.5 0.5 0.5 1.0"/>
+		</material>
+		</visual>
+		<collision>
+		<origin xyz="0 0 0"/>
+		<geometry>
+			<box size="0.01 0.01 0.01"/>
+		</geometry>
+		</collision>
+		<inertial>
+		<origin xyz="0 0 0" rpy="0 0 0"/>
+		<mass value="1e-6"/>
+		<inertia ixx="1e-6" ixy="0" ixz="0"
+				iyy="1e-6" iyz="0"
+				izz="1e-6"/>
+		</inertial>
+	</link>
+	<!-- os_sensor frame {{{ -->
+	<joint name="os_sensor_joint" type="fixed">
+		<parent link="mst110cr_2/os_stand"/>
+		<child link="mst110cr_2/os_sensor"/>
+		<origin xyz="0.040 0.000 0.085" rpy="0 0 0"/>
+	</joint>
+	<link name="mst110cr_2/os_sensor">
+		<visual>
+		<origin xyz="0 0 0"/>
+		<geometry>
+			<box size="0.01 0.01 0.01"/>
+		</geometry>
+		<material name="gray">
+			<color rgba="0.5 0.5 0.5 1.0"/>
+		</material>
+		</visual>
+		<collision>
+		<origin xyz="0 0 0"/>
+		<geometry>
+			<box size="0.01 0.01 0.01"/>
+		</geometry>
+		</collision>
+		<inertial>
+		<origin xyz="0 0 0" rpy="0 0 0"/>
+		<mass value="1e-6"/>
+		<inertia ixx="1e-6" ixy="0" ixz="0"
+				iyy="1e-6" iyz="0"
+				izz="1e-6"/>
+		</inertial>
+	</link>
+	<!-- livox_fr frame {{{ -->
+	<joint name="livox_fr_joint" type="fixed">
+		<parent link="mst110cr_2/body_link"/>
+		<child link="mst110cr_2/livox_fr"/>
+		<origin xyz="2.98 -1.4 0.2" rpy="${radians(180)} 0 0"/>
+	</joint>
+	<link name="mst110cr_2/livox_fr">
+		<visual>
+		<origin xyz="0 0 0"/>
+		<geometry>
+			<box size="0.01 0.01 0.01"/>
+		</geometry>
+		<material name="gray">
+			<color rgba="0.5 0.5 0.5 1.0"/>
+		</material>
+		</visual>
+		<collision>
+		<origin xyz="0 0 0"/>
+		<geometry>
+			<box size="0.01 0.01 0.01"/>
+		</geometry>
+		</collision>
+		<inertial>
+		<origin xyz="0 0 0" rpy="0 0 0"/>
+		<mass value="1e-6"/>
+		<inertia ixx="1e-6" ixy="0" ixz="0"
+				iyy="1e-6" iyz="0"
+				izz="1e-6"/>
+		</inertial>
+	</link>
+	<!-- livox_fl frame {{{ -->
+	<joint name="livox_fl_joint" type="fixed">
+		<parent link="mst110cr_2/body_link"/>
+		<child link="mst110cr_2/livox_fl"/>
+		<origin xyz="2.98 1.4 0.2" rpy="${radians(180)} 0 0"/>
+	</joint>
+	<link name="mst110cr_2/livox_fl">
+		<visual>
+		<origin xyz="0 0 0"/>
+		<geometry>
+			<box size="0.01 0.01 0.01"/>
+		</geometry>
+		<material name="gray">
+			<color rgba="0.5 0.5 0.5 1.0"/>
+		</material>
+		</visual>
+		<collision>
+		<origin xyz="0 0 0"/>
+		<geometry>
+			<box size="0.01 0.01 0.01"/>
+		</geometry>
+		</collision>
+		<inertial>
+		<origin xyz="0 0 0" rpy="0 0 0"/>
+		<mass value="1e-6"/>
+		<inertia ixx="1e-6" ixy="0" ixz="0"
+				iyy="1e-6" iyz="0"
+				izz="1e-6"/>
+		</inertial>
+	</link>
+	<!-- livox_rr frame {{{ -->
+	<joint name="livox_rr_joint" type="fixed">
+		<parent link="mst110cr_2/body_link"/>
+		<child link="mst110cr_2/livox_rr"/>
+		<origin xyz="-2.4 -0.555 0.2" rpy="${radians(180)} 0 ${radians(180)}"/>
+	</joint>
+	<link name="mst110cr_2/livox_rr">
+		<visual>
+		<origin xyz="0 0 0"/>
+		<geometry>
+			<box size="0.01 0.01 0.01"/>
+		</geometry>
+		<material name="gray">
+			<color rgba="0.5 0.5 0.5 1.0"/>
+		</material>
+		</visual>
+		<collision>
+		<origin xyz="0 0 0"/>
+		<geometry>
+			<box size="0.01 0.01 0.01"/>
+		</geometry>
+		</collision>
+		<inertial>
+		<origin xyz="0 0 0" rpy="0 0 0"/>
+		<mass value="1e-6"/>
+		<inertia ixx="1e-6" ixy="0" ixz="0"
+				iyy="1e-6" iyz="0"
+				izz="1e-6"/>
+		</inertial>
+	</link>
+	<!-- livox_rl frame {{{ -->
+	<joint name="livox_rl_joint" type="fixed">
+		<parent link="mst110cr_2/body_link"/>
+		<child link="mst110cr_2/livox_rl"/>
+		<origin xyz="-2.4 0.555 0.2" rpy="${radians(180)} 0 ${radians(180)}"/>
+	</joint>
+	<link name="mst110cr_2/livox_rl">
+		<visual>
+		<origin xyz="0 0 0"/>
+		<geometry>
+			<box size="0.01 0.01 0.01"/>
+		</geometry>
+		<material name="gray">
+			<color rgba="0.5 0.5 0.5 1.0"/>
+		</material>
+		</visual>
+		<collision>
+		<origin xyz="0 0 0"/>
+		<geometry>
+			<box size="0.01 0.01 0.01"/>
+		</geometry>
+		</collision>
+		<inertial>
+		<origin xyz="0 0 0" rpy="0 0 0"/>
+		<mass value="1e-6"/>
+		<inertia ixx="1e-6" ixy="0" ixz="0"
+				iyy="1e-6" iyz="0"
+				izz="1e-6"/>
+		</inertial>
+	</link>
 	<!-- Vessel {{{ -->
 	<joint name="vessel_pin_joint" type="revolute">

Commit message: Add: unity上のmst110crのナビゲーション機能を追加開発

File: mst110cr_description/urdf/mst110cr.xacro (robot description, xacro)
@@ -2,11 +2,14 @@
 <robot name="mst110cr" xmlns:xacro="http://www.ros.org/wiki/xacro">
 	<!-- Base Link -->
-	<link name="mst110cr_2/base_link"/>
+  <xacro:arg name="prefix" default="mst110cr_2"/>
+  <xacro:property name="prefix" value="$(arg prefix)"/>
+  <xacro:arg name="prefix" default="mst110cr_2"/>
+	<link name="${prefix}/base_link"/>
 	<!-- Track {{{ -->
 	<joint name="base_joint" type="fixed">
-		<parent link="mst110cr_2/base_link"/>
-		<child link="mst110cr_2/track_link"/>
+		<parent link="${prefix}/base_link"/>
+		<child link="${prefix}/track_link"/>
 	</joint>
-	<link name="mst110cr_2/track_link">
+	<link name="${prefix}/track_link">
 		<visual>
 			<geometry>
@@ -32,8 +35,8 @@
 		<origin xyz="0 0 1"/>
 		<axis xyz="0 0 1"/>
-		<parent link="mst110cr_2/track_link"/>
-		<child link="mst110cr_2/body_link"/>
+		<parent link="${prefix}/track_link"/>
+		<child link="${prefix}/body_link"/>
 	</joint>
-	<link name="mst110cr_2/body_link">
+	<link name="${prefix}/body_link">
 		<visual>
 			<origin xyz="0 0 0"/>
@@ -61,9 +64,9 @@
 		<origin xyz="-2.389 0 0.562"/>
 		<axis xyz="0 1 0"/>
-		<parent link="mst110cr_2/body_link"/>
-		<child link="mst110cr_2/vessel_link"/>
+		<parent link="${prefix}/body_link"/>
+		<child link="${prefix}/vessel_link"/>
 		<limit lower="${radians(-60)}" upper="${radians(0)}" effort="500" velocity="6.159937255"/>
 	</joint>
-	<link name="mst110cr_2/vessel_link">
+	<link name="${prefix}/vessel_link">
 		<visual>
 			<origin xyz="0 0 0"/>
@@ -91,9 +94,9 @@
 		<origin xyz="-1.891 0 0.293"/>
 		<axis xyz="0 1 0"/>
-		<parent link="mst110cr_2/body_link"/>
-		<child link="mst110cr_2/vessel_cylinder_link"/>
+		<parent link="${prefix}/body_link"/>
+		<child link="${prefix}/vessel_cylinder_link"/>
 		<mimic joint="vessel_pin_joint" multiplier="${66/60}"/>
 	</joint>
-	<link name="mst110cr_2/vessel_cylinder_link">
+	<link name="${prefix}/vessel_cylinder_link">
 		<visual>
 			<origin xyz="0 0 0"/>
@@ -121,10 +124,10 @@
 		<origin xyz="0 0 0"/>
 		<axis xyz="1.039 0 0.282"/>
-		<parent link="mst110cr_2/vessel_cylinder_link"/>
-		<child link="mst110cr_2/vessel_rod_link"/>
+		<parent link="${prefix}/vessel_cylinder_link"/>
+		<child link="${prefix}/vessel_rod_link"/>
 		<limit lower="0" upper="0.6" effort="500" velocity="6.159937255"/>
 		<mimic joint="vessel_pin_joint" multiplier="${0.6/radians(-60)}"/>
 	</joint>
-	<link name="mst110cr_2/vessel_rod_link">
+	<link name="${prefix}/vessel_rod_link">
 		<visual>
 			<origin xyz="0 0 0"/>
@@ -151,7 +154,7 @@
 		<origin xyz="1.42 0.60 2.20"/>
 		<axis xyz="0 0 1"/>
-		<parent link="mst110cr_2/body_link"/>
-		<child link="mst110cr_2/gnss_link"/>
+		<parent link="${prefix}/body_link"/>
+		<child link="${prefix}/gnss_link"/>
 	</joint>
-	<link name="mst110cr_2/gnss_link"/>
+	<link name="${prefix}/gnss_link"/>
 </robot>

Commit message: Update: パラメータをチューニング + physxからのメッセージ内容のミスを修正するノードを追加

File: mst110cr_description/urdf/mst110cr.xacro (robot description, xacro)
@@ -4,5 +4,4 @@
   <xacro:arg name="prefix" default="mst110cr_2"/>
   <xacro:property name="prefix" value="$(arg prefix)"/>
-  <xacro:arg name="prefix" default="mst110cr_2"/>
 	<link name="${prefix}/base_link"/>
 	<!-- Track {{{ -->
@@ -32,5 +31,5 @@
 	<!-- }}} Track ends here -->
 	<!-- Body {{{ -->
-	<joint name="swing_joint" type="continuous">
+	<joint name="rotate_joint" type="continuous">
 		<origin xyz="0 0 1"/>
 		<axis xyz="0 0 1"/>
